Commit message: revision code at 2nd day class from linux

File: week_11_Simulation_Basic/robot_description/urdf/robot.urdf (robot description, URDF)
Before this commit: robot robot, 3 links, 2 joints
Links:
- added link link_caster_wheel, mass 1; collision sphere radius=0.10; collision sphere radius=0.2
- link link_chassis: geometry collision box size=2 1.3 0.4; visual box size=2 1.3 0.4
- link link_left_wheel: geometry collision cylinder length=0.12 radius=0.08; collision cylinder length=0.12 radius=0.4
- link link_right_wheel: geometry collision cylinder length=0.12 radius=0.08; collision cylinder length=0.12 radius=0.4
Joints:
- added joint joint_chassis_caster_wheel: type fixed, parent link_chassis, child link_caster_wheel, origin xyz=0.8 0 -0.15 rpy=0 0 0

File: week_11_Simulation_Basic/robot_description/urdf/robot_mesh.urdf (robot description, URDF)
Before this commit: robot robot, 3 links, 2 joints
Links:
- added link link_caster_wheel, mass 1; collision sphere radius=0.10; collision sphere radius=0.2
- link link_chassis: geometry collision mesh filename=package://robot_description/meshes/chassis.stl; visual mesh filename=package://robot_description/meshes/chassis.stl
- link link_left_wheel: geometry collision cylinder length=0.12 radius=0.08; collision cylinder length=0.12 radius=0.4
- link link_right_wheel: geometry collision cylinder length=0.12 radius=0.08; collision cylinder length=0.12 radius=0.4
Joints:
- added joint joint_chassis_caster_wheel: type fixed, parent link_chassis, child link_caster_wheel, origin xyz=0.8 0 -0.15 rpy=0 0 0

Commit message: final files to practice simulation basic

File: week_11_Simulation_Basic/robot_description/urdf/robot.urdf (robot description, URDF)
Before this commit: robot robot, 4 links, 3 joints
Links:
- added link link_laser_scan, mass 0.5; collision cylinder length=0.20 radius=0.15; visual cylinder length=0.20 radius=0.15
- link link_chassis: geometry collision mesh filename=package://robot_description/meshes/chassis.stl; visual mesh filename=package://robot_description/meshes/chassis.stl
- link link_left_wheel: geometry collision cylinder length=0.12 radius=0.08; collision cylinder length=0.12 radius=0.4
- link link_right_wheel: geometry collision cylinder length=0.12 radius=0.08; collision cylinder length=0.12 radius=0.4
Joints:
- added joint joint_laser_scan_chassis: type fixed, parent link_chassis, child link_laser_scan, origin xyz=0.8 0 0.3 rpy=0 0 0

File: week_11_Simulation_Basic/robot_description/urdf/robot.xacro (robot description, xacro)
@@ -226,44 +226,3 @@
         </collision>
     </link>
-    <!-- Robot tail -->
-    <joint name="joint_tail" type="continuous">
-        <origin rpy="0 0 0" xyz="-1 0 0" />
-        <child link="link_tail" />
-        <axis rpy="0 0 0" xyz="0 1 0" />
-        <parent link="link_chassis" />
-        <joint_properties damping="1.0" friction="1.0" />
-    </joint>
-    <link name="link_tail">
-        <inertial>
-            <origin xyz="0 0 0" rpy="0 0 0" />
-            <mass value="0.5" />
-            <inertia ixx="0.000252666666667" ixy="0" ixz="0" iyy="0.000252666666667" iyz="0" izz="0.0005"/>
-        </inertial>
-        <visual>
-            <origin xyz="-0.2 0 0" rpy="0 ${pi/2} 0" />
-            <geometry>
-                <cylinder radius="0.05" length="0.40"/>
-            </geometry>
-            <material name="Red">
-                <color rgba="0.7 0.1 0.1 1" />
-            </material>
-        </visual>
-        <collision>
-            <origin xyz="-0.2 0 0" rpy="0 ${pi/2} 0"/>
-            <geometry>
-                <cylinder radius="0.05" length="0.40"/>
-            </geometry>
-        </collision>
-    </link>
-    <!-- Transmission -->
-    <transmission name="tran_tail">
-        <type>transmission_interface/SimpleTransmission</type>
-        <joint name="joint_tail">
-            <hardwareInterface>hardware_interface/EffortJointInterface</hardwareInterface>
-        </joint>
-        <actuator name="motor_joint_tail">
-            <hardwareInterface>hardware_interface/EffortJointInterface</hardwareInterface>
-            <mechanicalReduction>1</mechanicalReduction>
-        </actuator>
-    </transmission>
 </robot>
